File: VersionControlTest/VersionControlTest.kicad_sch (KiCad schematic)
At the start: 0 parts

Commit message: add 2 R power
Parts:
- added R1: 100R, Resistor_SMD:R_0603_1608Metric, symbol Device:R
- added R2: 470R, Resistor_SMD:R_0603_1608Metric, symbol Device:R
Connections:
- new net +5V: R1.1, R2.1
- new net GND: R1.2, R2.2
